Commit message: temp fix gazebo crash due to collision

File: rover_system/model/MR_arm.urdf.xacro (robot description, xacro)
@@ -219,4 +219,19 @@
       </collision>
     </link>
+    <!-- Prevent crash in ign gazebo -->
+    <disable_collisions link1="link_1_waist_shoulder" link2="link_2_shoulder_elbow"
+      reason="Adjacent" />
+    <disable_collisions link1="link_2_shoulder_elbow" link2="link_3_elbow_wrist_pitch"
+      reason="Adjacent" />
+    <disable_collisions link1="link_3_elbow_wrist_pitch" link2="link_4_wrist_pitch_wrist_roll"
+      reason="Adjacent" />
+    <disable_collisions link1="link_4_wrist_pitch_wrist_roll" link2="link_5_wrist_roll_end_effector"
+      reason="Adjacent" />
+    <disable_collisions link1="link_5_wrist_roll_end_effector" link2="link_6_end_effector_1"
+      reason="Adjacent" />
+    <disable_collisions link1="link_5_wrist_roll_end_effector" link2="link_7_end_effector_2"
+      reason="Adjacent" />
+    <disable_collisions link1="link_6_end_effector_1" link2="link_7_end_effector_2"
+      reason="Adjacent" />
   </xacro:macro>
 </robot>

File: rover_system/model/rover.urdf.xacro (robot description, xacro)
@@ -24,5 +24,5 @@
                 <!-- <mesh
                     filename="file://$(find rover_system)/model/meshes/Full_Asm_Adjusted.dae" /> -->
-                <box size="0 0 0" />
+                <!-- <box size="1 1 1" /> -->
             </geometry>
         </collision>
@@ -57,7 +57,8 @@
         <origin xyz="0 -0.41 0.32" rpy="0 0 -1.57079" />
     </xacro:depth_camera> -->
-    <xacro:MR_arm parent_link="chassis_link">
+    <!-- TODO FIXME arm collision crashes gazebo -->
+    <!-- <xacro:MR_arm parent_link="chassis_link">
         <origin xyz="0 -0.28 ${0.37}" rpy="0 0 -1.57079" />
-    </xacro:MR_arm>
+    </xacro:MR_arm> -->
     <!-- Gazebo Plugins -->
     <gazebo>

Commit message: fixed xacro

File: rover_system/model/MR_arm.urdf.xacro (robot description, xacro)
@@ -37,4 +37,6 @@
         <origin xyz="0 0 0" rpy="0 0 0" />
         <inertia ixx="0" ixy="0" ixz="0" iyy="0" iyz="0" izz="0" />
+        <gravity>0</gravity>
+        <self_collide>1</self_collide>
       </inertial>
       <visual>
@@ -65,4 +67,6 @@
         <origin xyz="0 0 0" rpy="0 0 0" />
         <inertia ixx="0" ixy="0" ixz="0" iyy="0" iyz="0" izz="0" />
+        <gravity>0</gravity>
+        <self_collide>1</self_collide>
       </inertial>
       <visual>
@@ -93,4 +97,6 @@
         <origin xyz="0 0 0" rpy="0 0 0" />
         <inertia ixx="0" ixy="0" ixz="0" iyy="0" iyz="0" izz="0" />
+        <gravity>0</gravity>
+        <self_collide>1</self_collide>
       </inertial>
       <visual>
@@ -121,4 +127,6 @@
         <origin xyz="0 0 0" rpy="0 0 0" />
         <inertia ixx="0" ixy="0" ixz="0" iyy="0" iyz="0" izz="0" />
+        <gravity>0</gravity>
+        <self_collide>1</self_collide>
       </inertial>
       <visual>
@@ -149,4 +157,6 @@
         <origin xyz="0 0 0" rpy="0 0 0" />
         <inertia ixx="0" ixy="0" ixz="0" iyy="0" iyz="0" izz="0" />
+        <gravity>0</gravity>
+        <self_collide>1</self_collide>
       </inertial>
       <visual>

File: rover_system/model/wheel.urdf.xacro (robot description, xacro)
@@ -25,7 +25,8 @@
 			</visual>
 			<collision>
-				<origin xyz="0.03 0 0" rpy="0 ${M_PI/2} 0" />
+				<!-- <origin xyz="0.03 0 0" rpy="${M_PI/2} ${M_PI/2} 0" /> -->
+				<origin xyz="0 0 0" rpy="0 0 0" />
 				<geometry>
-					<cylinder length="0.2" radius="0.14" />
+					<cylinder length="0.2" radius="0.15" />
 				</geometry>
 			</collision>
