Commit message: debugging arm

File: rover_system/model/MR_arm_no_collision.urdf.xacro (robot description, xacro)
@@ -23,10 +23,10 @@
         </geometry>
       </visual>
-      <collision>
+      <!-- <collision>
         <origin xyz="0 0 0" rpy="0 0 0" />
         <geometry>
           <mesh filename="file://$(find rover_system)/model/meshes/collision_Link0.stl" />
         </geometry>
-      </collision>
+      </collision> -->
     </link>
     <joint name="joint_waist" type="revolute">
@@ -53,10 +53,10 @@
         </geometry>
       </visual>
-      <collision>
+      <!-- <collision>
         <origin xyz="0 0 0" rpy="0 0 0" />
         <geometry>
           <mesh filename="file://$(find rover_system)/model/meshes/collision_Link1.stl" />
         </geometry>
-      </collision>
+      </collision> -->
     </link>
     <joint
@@ -83,10 +83,10 @@
         </geometry>
       </visual>
-      <collision>
+      <!-- <collision>
         <origin xyz="0 0 0" rpy="0 0 0" />
         <geometry>
           <mesh filename="file://$(find rover_system)/model/meshes/collision_Link2.stl" />
         </geometry>
-      </collision>
+      </collision> -->
     </link>
     <joint
@@ -113,10 +113,10 @@
         </geometry>
       </visual>
-      <collision>
+      <!-- <collision>
         <origin xyz="0 0 0" rpy="0 0 0" />
         <geometry>
           <mesh filename="file://$(find rover_system)/model/meshes/collision_Link3.stl" />
         </geometry>
-      </collision>
+      </collision> -->
     </link>
     <joint
@@ -143,10 +143,10 @@
         </geometry>
       </visual>
-      <collision>
+      <!-- <collision>
         <origin xyz="0 0 0" rpy="0 0 0" />
         <geometry>
           <mesh filename="file://$(find rover_system)/model/meshes/collision_Link4.stl" />
         </geometry>
-      </collision>
+      </collision> -->
     </link>
     <joint
@@ -173,10 +173,10 @@
         </geometry>
       </visual>
-      <collision>
+      <!-- <collision>
         <origin xyz="0 0 0" rpy="0 0 0" />
         <geometry>
           <mesh filename="file://$(find rover_system)/model/meshes/collision_Link5.stl" />
         </geometry>
-      </collision>
+      </collision> -->
     </link>
     <joint
@@ -209,10 +209,10 @@
         </geometry>
       </visual>
-      <collision>
+      <!-- <collision>
         <origin xyz="0 0 0" rpy="0 0 0" />
         <geometry>
           <box size="0.1 0.1 0.1" />
         </geometry>
-      </collision>
+      </collision> -->
     </link>
     <link
@@ -229,10 +229,10 @@
         </geometry>
       </visual>
-      <collision>
+      <!-- <collision>
         <origin xyz="0 0 0" rpy="0 0 0" />
         <geometry>
           <box size="0.1 0.1 0.1" />
         </geometry>
-      </collision>
+      </collision> -->
     </link>
     <!-- Prevent crash in ign gazebo -->

File: rover_system/model/rover.urdf.xacro (robot description, xacro)
@@ -58,7 +58,7 @@
     </xacro:depth_camera> -->
     <!-- TODO FIXME arm collision crashes gazebo -->
-    <!-- <xacro:MR_arm parent_link="chassis_link">
+    <xacro:MR_arm parent_link="chassis_link">
         <origin xyz="0 -0.28 ${0.37}" rpy="0 0 -1.57079" />
-    </xacro:MR_arm> -->
+    </xacro:MR_arm>
     <!-- Gazebo Plugins -->
     <gazebo>
