Commit message: fix rover model wheel offset and add arm

File: rover_system/model/rover.urdf.xacro (robot description, xacro)
@@ -2,8 +2,10 @@
     <!-- Robot Parameters -->
     <xacro:property name="chassis_mass" value="45.2" />
+    <xacro:property name="pi_constant" value="3.14159" />
+    <xacro:property name="wheel_z_offset" value="${-0.060752 + 0.1 * 2}" />
     <!-- Part Includes - Payload, Sensors, Etc.. -->
     <xacro:include filename="$(find rover_system)/model/wheel.urdf.xacro" />
-    <!-- <xacro:include filename="$(find rover_system)/model/depth_camera.urdf.xacro" />a
-    <xacro:include filename="$(find rover_system)/model/MR_arm.urdf.xacro" /> -->
+    <!-- <xacro:include filename="$(find rover_system)/model/depth_camera.urdf.xacro" />a -->
+    <xacro:include filename="$(find rover_system)/model/MR_arm.urdf.xacro" />
     <xacro:include filename="$(find rover_system)/model/imu.urdf" />
     <!-- Robot Definition -->
@@ -41,21 +43,21 @@
     <!-- Wheels -->
     <xacro:wheel wheel_prefix="lf" parent_link="base_link">
-        <origin xyz="0.5125 -0.316275 ${-0.060752 + .1}" rpy="0 1.57079 0" />
+        <origin xyz="0.5125 -0.316275 ${wheel_z_offset}" rpy="0 0 0" />
     </xacro:wheel>
     <xacro:wheel wheel_prefix="rf" parent_link="base_link">
-        <origin xyz="-0.5125 -0.316275 ${-0.060752 + .1}" rpy="0 1.57079 0" />
+        <origin xyz="-0.5125 -0.316275 ${wheel_z_offset}" rpy="0 0 0" />
     </xacro:wheel>
     <xacro:wheel wheel_prefix="lb" parent_link="base_link">
-        <origin xyz="0.5125 0.306875 ${-0.060752 + .1}" rpy="0 1.57079 0" />
+        <origin xyz="0.5125 0.306875 ${wheel_z_offset}" rpy="0 0 0" />
     </xacro:wheel>
     <xacro:wheel wheel_prefix="rb" parent_link="base_link">
-        <origin xyz="-0.5125 0.306875 ${-0.060752 + .1}" rpy="0 1.57079 0" />
+        <origin xyz="-0.5125 0.306875 ${wheel_z_offset}" rpy="0 0 0" />
     </xacro:wheel>
     <!-- <xacro:depth_camera parent_link="base_link">
         <origin xyz="0 -0.41 0.32" rpy="0 0 -1.57079" />
-    </xacro:depth_camera>
+    </xacro:depth_camera> -->
     <xacro:MR_arm parent_link="base_link">
-        <origin xyz="0 -0.28 0.37" rpy="0 0 -1.57079" />
-    </xacro:MR_arm> -->
+        <origin xyz="0 -0.28 ${0.37}" rpy="0 0 -1.57079" />
+    </xacro:MR_arm>
     <!-- Gazebo Plugins -->
     <gazebo>

Commit message: updated new meshes

File: rover_system/model/rover.urdf.xacro (robot description, xacro)
@@ -2,6 +2,6 @@
     <!-- Robot Parameters -->
     <xacro:property name="chassis_mass" value="45.2" />
-    <xacro:property name="pi_constant" value="3.14159" />
-    <xacro:property name="wheel_z_offset" value="${-0.060752 + 0.1 * 2}" />
+    <xacro:property name="M_PI" value="3.14159265" />
+    <xacro:property name="wheel_z_offset" value="${-0.060752 + 0.1}" />
     <!-- Part Includes - Payload, Sensors, Etc.. -->
     <xacro:include filename="$(find rover_system)/model/wheel.urdf.xacro" />
@@ -16,5 +16,5 @@
             <geometry>
                 <mesh
-                    filename="file://$(find rover_system)/model/meshes/Full_Asm_Adjusted.dae" />
+                    filename="file://$(find rover_system)/model/meshes/Full_Asm_noarm_mast_cam.dae" />
             </geometry>
         </visual>
@@ -22,7 +22,7 @@
             <origin xyz="0 0 0.1" rpy="0 0 0" />
             <geometry>
-                <mesh
-                    filename="file://$(find rover_system)/model/meshes/Full_Asm_Adjusted.dae" />
-                <!-- <box size="0 0 0" /> -->
+                <!-- <mesh
+                    filename="file://$(find rover_system)/model/meshes/Full_Asm_Adjusted.dae" /> -->
+                <box size="0 0 0" />
             </geometry>
         </collision>
@@ -39,23 +39,23 @@
         <parent link="base_link" />
         <child link="chassis_link" />
-        <origin xyz="0 0 0.125" />
+        <origin xyz="0 0 0" />
     </joint>
     <!-- Wheels -->
-    <xacro:wheel wheel_prefix="lf" parent_link="base_link">
-        <origin xyz="0.5125 -0.316275 ${wheel_z_offset}" rpy="0 0 0" />
+    <xacro:wheel wheel_prefix="lf" parent_link="chassis_link">
+        <origin xyz="0.5125 -0.316275 ${wheel_z_offset}" rpy="0 ${M_PI/2} 0" />
     </xacro:wheel>
-    <xacro:wheel wheel_prefix="rf" parent_link="base_link">
-        <origin xyz="-0.5125 -0.316275 ${wheel_z_offset}" rpy="0 0 0" />
+    <xacro:wheel wheel_prefix="rf" parent_link="chassis_link">
+        <origin xyz="-0.5125 -0.316275 ${wheel_z_offset}" rpy="0 ${M_PI/2} 0" />
     </xacro:wheel>
-    <xacro:wheel wheel_prefix="lb" parent_link="base_link">
-        <origin xyz="0.5125 0.306875 ${wheel_z_offset}" rpy="0 0 0" />
+    <xacro:wheel wheel_prefix="lb" parent_link="chassis_link">
+        <origin xyz="0.5125 0.306875 ${wheel_z_offset}" rpy="0 ${M_PI/2} 0" />
     </xacro:wheel>
-    <xacro:wheel wheel_prefix="rb" parent_link="base_link">
-        <origin xyz="-0.5125 0.306875 ${wheel_z_offset}" rpy="0 0 0" />
+    <xacro:wheel wheel_prefix="rb" parent_link="chassis_link">
+        <origin xyz="-0.5125 0.306875 ${wheel_z_offset}" rpy="0 ${M_PI/2} 0" />
     </xacro:wheel>
-    <!-- <xacro:depth_camera parent_link="base_link">
+    <!-- <xacro:depth_camera parent_link="chassis_link">
         <origin xyz="0 -0.41 0.32" rpy="0 0 -1.57079" />
     </xacro:depth_camera> -->
-    <xacro:MR_arm parent_link="base_link">
+    <xacro:MR_arm parent_link="chassis_link">
         <origin xyz="0 -0.28 ${0.37}" rpy="0 0 -1.57079" />
     </xacro:MR_arm>

File: rover_system/model/wheel.urdf.xacro (robot description, xacro)
@@ -21,5 +21,5 @@
 				<geometry>
 					<mesh
-						filename="file://$(find rover_system)/model/meshes/full_wheel_assembly_fixed.dae" />
+						filename="file://$(find rover_system)/model/meshes/WHEEL.dae" />
 				</geometry>
 			</visual>

Commit message: fixed typo in xacro

File: rover_system/model/rover.urdf.xacro (robot description, xacro)
@@ -39,5 +39,5 @@
         <parent link="base_link" />
         <child link="chassis_link" />
-        <origin xyz="0 0 0" />
+        <origin xyz="0 0 0.2" />
     </joint>
     <!-- Wheels -->
@@ -69,6 +69,6 @@
             <!-- Wheel Information -->
             <left_joint>lf_wheel</left_joint>
-            <left_joint>rf_wheel</left_joint>
-            <right_joint>lb_wheel</right_joint>
+            <left_joint>lb_wheel</left_joint>
+            <right_joint>rf_wheel</right_joint>
             <right_joint>rb_wheel</right_joint>
             <wheel_separation>0.63255</wheel_separation>

File: rover_system/model/wheel.urdf.xacro (robot description, xacro)
@@ -36,15 +36,15 @@
 			<child link="${wheel_prefix}_wheel_link" />
 			<xacro:insert_block name="joint_pose" />
-			<xacro:if value="${wheel_prefix == 'left'}">
-				<axis xyz="-1 0 0" rpy="0 0 0" />
+			<xacro:if value="${wheel_prefix == 'lf'}">
+				<axis xyz="0 0 1" />
 			</xacro:if>
-			<xacro:if value="${wheel_prefix == 'right'}">
-				<axis xyz="1 0 0" rpy="0 0 0" />
+			<xacro:if value="${wheel_prefix == 'rf'}">
+				<axis xyz="0 0 1" />
 			</xacro:if>
-			<xacro:if value="${wheel_prefix == 'rear_left'}">
-				<axis xyz="-1 0 0" rpy="0 0 0" />
+			<xacro:if value="${wheel_prefix == 'lb'}">
+				<axis xyz="0 0 1" />
 			</xacro:if>
-			<xacro:if value="${wheel_prefix == 'rear_right'}">
-				<axis xyz="1 0 0" rpy="0 0 0" />
+			<xacro:if value="${wheel_prefix == 'rb'}">
+				<axis xyz="0 0 1" />
 			</xacro:if>
 			<limit effort="300" velocity="50.0" />

Commit message: fix collision box

File: rover_system/model/rover.urdf.xacro (robot description, xacro)
@@ -20,9 +20,9 @@
         </visual>
         <collision>
-            <origin xyz="0 0 0.1" rpy="0 0 0" />
+            <origin xyz="0 0 0.2" rpy="0 0 0" />
             <geometry>
                 <!-- <mesh
                     filename="file://$(find rover_system)/model/meshes/Full_Asm_Adjusted.dae" /> -->
-                <!-- <box size="1 1 1" /> -->
+                <box size="0.4 0.6 0.3" />
             </geometry>
         </collision>

Commit message: fixup! fix collision box

File: rover_system/model/rover.urdf.xacro (robot description, xacro)
@@ -33,5 +33,6 @@
             <!-- <inertia ixx="1.7724" ixy="0.0" ixz="0.0" iyy="0.141558" iyz="-0.0" izz="0.179826"
             /> -->
-            <inertia ixx="0.0" ixy="0.0" ixz="0.0" iyy="0.0" iyz="0.0" izz="0.0" />
+            <!-- <inertia ixx="0.0" ixy="0.0" ixz="0.0" iyy="0.0" iyz="0.0" izz="0.0" /> -->
+            <inertia ixx="1.3569" ixy="0.0" ixz="0.0" iyy="1.924" iyz="0.0" izz="0.847" />
         </inertial>
     </link>
