Commit message: folder structure

File: sim/model/MR_arm.urdf.xacro (robot description, xacro)
@@ -20,11 +20,11 @@
         <origin xyz="0 0 0" rpy="0 0 0" />
         <geometry>
-          <mesh filename="file://$(find rover_system)/model/meshes/Link0.stl" />
-        </geometry>
-      </visual>
-      <collision>
-        <origin xyz="0 0 0" rpy="0 0 0" />
-        <geometry>
-          <mesh filename="file://$(find rover_system)/model/meshes/collision_Link0.stl" />
+          <mesh filename="file://$(find sim)/model/meshes/Link0.stl" />
+        </geometry>
+      </visual>
+      <collision>
+        <origin xyz="0 0 0" rpy="0 0 0" />
+        <geometry>
+          <mesh filename="file://$(find sim)/model/meshes/collision_Link0.stl" />
         </geometry>
       </collision>
@@ -50,11 +50,11 @@
         <origin xyz="0 0 0" rpy="0 0 0" />
         <geometry>
-          <mesh filename="file://$(find rover_system)/model/meshes/Link1.stl" />
-        </geometry>
-      </visual>
-      <collision>
-        <origin xyz="0 0 0" rpy="0 0 0" />
-        <geometry>
-          <mesh filename="file://$(find rover_system)/model/meshes/collision_Link1.stl" />
+          <mesh filename="file://$(find sim)/model/meshes/Link1.stl" />
+        </geometry>
+      </visual>
+      <collision>
+        <origin xyz="0 0 0" rpy="0 0 0" />
+        <geometry>
+          <mesh filename="file://$(find sim)/model/meshes/collision_Link1.stl" />
         </geometry>
       </collision>
@@ -80,11 +80,11 @@
         <origin xyz="0 0 0" rpy="0 0 0" />
         <geometry>
-          <mesh filename="file://$(find rover_system)/model/meshes/Link2.stl" />
-        </geometry>
-      </visual>
-      <collision>
-        <origin xyz="0 0 0" rpy="0 0 0" />
-        <geometry>
-          <mesh filename="file://$(find rover_system)/model/meshes/collision_Link2.stl" />
+          <mesh filename="file://$(find sim)/model/meshes/Link2.stl" />
+        </geometry>
+      </visual>
+      <collision>
+        <origin xyz="0 0 0" rpy="0 0 0" />
+        <geometry>
+          <mesh filename="file://$(find sim)/model/meshes/collision_Link2.stl" />
         </geometry>
       </collision>
@@ -110,11 +110,11 @@
         <origin xyz="0 0 0" rpy="0 0 0" />
         <geometry>
-          <mesh filename="file://$(find rover_system)/model/meshes/Link3.stl" />
-        </geometry>
-      </visual>
-      <collision>
-        <origin xyz="0 0 0" rpy="0 0 0" />
-        <geometry>
-          <mesh filename="file://$(find rover_system)/model/meshes/collision_Link3.stl" />
+          <mesh filename="file://$(find sim)/model/meshes/Link3.stl" />
+        </geometry>
+      </visual>
+      <collision>
+        <origin xyz="0 0 0" rpy="0 0 0" />
+        <geometry>
+          <mesh filename="file://$(find sim)/model/meshes/collision_Link3.stl" />
         </geometry>
       </collision>
@@ -140,11 +140,11 @@
         <origin xyz="0 0 0" rpy="0 0 0" />
         <geometry>
-          <mesh filename="file://$(find rover_system)/model/meshes/Link4.stl" />
-        </geometry>
-      </visual>
-      <collision>
-        <origin xyz="0 0 0" rpy="0 0 0" />
-        <geometry>
-          <mesh filename="file://$(find rover_system)/model/meshes/collision_Link4.stl" />
+          <mesh filename="file://$(find sim)/model/meshes/Link4.stl" />
+        </geometry>
+      </visual>
+      <collision>
+        <origin xyz="0 0 0" rpy="0 0 0" />
+        <geometry>
+          <mesh filename="file://$(find sim)/model/meshes/collision_Link4.stl" />
         </geometry>
       </collision>
@@ -170,11 +170,11 @@
         <origin xyz="0 0 0" rpy="0 0 0" />
         <geometry>
-          <mesh filename="file://$(find rover_system)/model/meshes/Link5.stl" />
-        </geometry>
-      </visual>
-      <collision>
-        <origin xyz="0 0 0" rpy="0 0 0" />
-        <geometry>
-          <mesh filename="file://$(find rover_system)/model/meshes/collision_Link5.stl" />
+          <mesh filename="file://$(find sim)/model/meshes/Link5.stl" />
+        </geometry>
+      </visual>
+      <collision>
+        <origin xyz="0 0 0" rpy="0 0 0" />
+        <geometry>
+          <mesh filename="file://$(find sim)/model/meshes/collision_Link5.stl" />
         </geometry>
       </collision>
@@ -206,5 +206,5 @@
         <origin xyz="0 0 0" rpy="0 0 0" />
         <geometry>
-          <mesh filename="file://$(find rover_system)/model/meshes/finger.stl" />
+          <mesh filename="file://$(find sim)/model/meshes/finger.stl" />
         </geometry>
       </visual>
@@ -226,5 +226,5 @@
         <origin xyz="0 0 0" rpy="0 0 0" />
         <geometry>
-          <mesh filename="file://$(find rover_system)/model/meshes/finger.stl" />
+          <mesh filename="file://$(find sim)/model/meshes/finger.stl" />
         </geometry>
       </visual>

File: sim/model/MR_arm_no_collision.urdf.xacro (robot description, xacro)
@@ -20,11 +20,11 @@
         <origin xyz="0 0 0" rpy="0 0 0" />
         <geometry>
-          <mesh filename="file://$(find rover_system)/model/meshes/Link0.stl" />
-        </geometry>
-      </visual>
-      <!-- <collision>
-        <origin xyz="0 0 0" rpy="0 0 0" />
-        <geometry>
-          <mesh filename="file://$(find rover_system)/model/meshes/collision_Link0.stl" />
+          <mesh filename="file://$(find sim)/model/meshes/Link0.stl" />
+        </geometry>
+      </visual>
+      <!-- <collision>
+        <origin xyz="0 0 0" rpy="0 0 0" />
+        <geometry>
+          <mesh filename="file://$(find sim)/model/meshes/collision_Link0.stl" />
         </geometry>
       </collision> -->
@@ -50,11 +50,11 @@
         <origin xyz="0 0 0" rpy="0 0 0" />
         <geometry>
-          <mesh filename="file://$(find rover_system)/model/meshes/Link1.stl" />
-        </geometry>
-      </visual>
-      <!-- <collision>
-        <origin xyz="0 0 0" rpy="0 0 0" />
-        <geometry>
-          <mesh filename="file://$(find rover_system)/model/meshes/collision_Link1.stl" />
+          <mesh filename="file://$(find sim)/model/meshes/Link1.stl" />
+        </geometry>
+      </visual>
+      <!-- <collision>
+        <origin xyz="0 0 0" rpy="0 0 0" />
+        <geometry>
+          <mesh filename="file://$(find sim)/model/meshes/collision_Link1.stl" />
         </geometry>
       </collision> -->
@@ -80,11 +80,11 @@
         <origin xyz="0 0 0" rpy="0 0 0" />
         <geometry>
-          <mesh filename="file://$(find rover_system)/model/meshes/Link2.stl" />
-        </geometry>
-      </visual>
-      <!-- <collision>
-        <origin xyz="0 0 0" rpy="0 0 0" />
-        <geometry>
-          <mesh filename="file://$(find rover_system)/model/meshes/collision_Link2.stl" />
+          <mesh filename="file://$(find sim)/model/meshes/Link2.stl" />
+        </geometry>
+      </visual>
+      <!-- <collision>
+        <origin xyz="0 0 0" rpy="0 0 0" />
+        <geometry>
+          <mesh filename="file://$(find sim)/model/meshes/collision_Link2.stl" />
         </geometry>
       </collision> -->
@@ -110,11 +110,11 @@
         <origin xyz="0 0 0" rpy="0 0 0" />
         <geometry>
-          <mesh filename="file://$(find rover_system)/model/meshes/Link3.stl" />
-        </geometry>
-      </visual>
-      <!-- <collision>
-        <origin xyz="0 0 0" rpy="0 0 0" />
-        <geometry>
-          <mesh filename="file://$(find rover_system)/model/meshes/collision_Link3.stl" />
+          <mesh filename="file://$(find sim)/model/meshes/Link3.stl" />
+        </geometry>
+      </visual>
+      <!-- <collision>
+        <origin xyz="0 0 0" rpy="0 0 0" />
+        <geometry>
+          <mesh filename="file://$(find sim)/model/meshes/collision_Link3.stl" />
         </geometry>
       </collision> -->
@@ -140,11 +140,11 @@
         <origin xyz="0 0 0" rpy="0 0 0" />
         <geometry>
-          <mesh filename="file://$(find rover_system)/model/meshes/Link4.stl" />
-        </geometry>
-      </visual>
-      <!-- <collision>
-        <origin xyz="0 0 0" rpy="0 0 0" />
-        <geometry>
-          <mesh filename="file://$(find rover_system)/model/meshes/collision_Link4.stl" />
+          <mesh filename="file://$(find sim)/model/meshes/Link4.stl" />
+        </geometry>
+      </visual>
+      <!-- <collision>
+        <origin xyz="0 0 0" rpy="0 0 0" />
+        <geometry>
+          <mesh filename="file://$(find sim)/model/meshes/collision_Link4.stl" />
         </geometry>
       </collision> -->
@@ -170,11 +170,11 @@
         <origin xyz="0 0 0" rpy="0 0 0" />
         <geometry>
-          <mesh filename="file://$(find rover_system)/model/meshes/Link5.stl" />
-        </geometry>
-      </visual>
-      <!-- <collision>
-        <origin xyz="0 0 0" rpy="0 0 0" />
-        <geometry>
-          <mesh filename="file://$(find rover_system)/model/meshes/collision_Link5.stl" />
+          <mesh filename="file://$(find sim)/model/meshes/Link5.stl" />
+        </geometry>
+      </visual>
+      <!-- <collision>
+        <origin xyz="0 0 0" rpy="0 0 0" />
+        <geometry>
+          <mesh filename="file://$(find sim)/model/meshes/collision_Link5.stl" />
         </geometry>
       </collision> -->
@@ -206,5 +206,5 @@
         <origin xyz="0 0 0" rpy="0 0 0" />
         <geometry>
-          <mesh filename="file://$(find rover_system)/model/meshes/finger.stl" />
+          <mesh filename="file://$(find sim)/model/meshes/finger.stl" />
         </geometry>
       </visual>
@@ -226,5 +226,5 @@
         <origin xyz="0 0 0" rpy="0 0 0" />
         <geometry>
-          <mesh filename="file://$(find rover_system)/model/meshes/finger.stl" />
+          <mesh filename="file://$(find sim)/model/meshes/finger.stl" />
         </geometry>
       </visual>

File: sim/model/MR_arm_seb.urdf.xacro (robot description, xacro)
@@ -19,11 +19,11 @@
         <origin xyz="0 0 0" rpy="0 0 0" />
         <geometry>
-          <mesh filename="file://$(find rover_system)/model/meshes/Link0.stl" />
-        </geometry>
-      </visual>
-      <collision>
-        <origin xyz="0 0 0" rpy="0 0 0" />
-        <geometry>
-          <mesh filename="file://$(find rover_system)/model/meshes/collision_Link0.stl" />
+          <mesh filename="file://$(find sim)/model/meshes/Link0.stl" />
+        </geometry>
+      </visual>
+      <collision>
+        <origin xyz="0 0 0" rpy="0 0 0" />
+        <geometry>
+          <mesh filename="file://$(find sim)/model/meshes/collision_Link0.stl" />
         </geometry>
       </collision>
@@ -49,11 +49,11 @@
         <origin xyz="0 0 0" rpy="0 0 0" />
         <geometry>
-          <mesh filename="file://$(find rover_system)/model/meshes/Link1.stl" />
-        </geometry>
-      </visual>
-      <collision>
-        <origin xyz="0 0 0" rpy="0 0 0" />
-        <geometry>
-          <mesh filename="file://$(find rover_system)/model/meshes/collision_Link1.stl" />
+          <mesh filename="file://$(find sim)/model/meshes/Link1.stl" />
+        </geometry>
+      </visual>
+      <collision>
+        <origin xyz="0 0 0" rpy="0 0 0" />
+        <geometry>
+          <mesh filename="file://$(find sim)/model/meshes/collision_Link1.stl" />
         </geometry>
       </collision>
@@ -78,11 +78,11 @@
         <origin xyz="0 0 0" rpy="0 0 0" />
         <geometry>
-          <mesh filename="file://$(find rover_system)/model/meshes/Link2.stl" />
-        </geometry>
-      </visual>
-      <collision>
-        <origin xyz="0 0 0" rpy="0 0 0" />
-        <geometry>
-          <mesh filename="file://$(find rover_system)/model/meshes/collision_Link2.stl" />
+          <mesh filename="file://$(find sim)/model/meshes/Link2.stl" />
+        </geometry>
+      </visual>
+      <collision>
+        <origin xyz="0 0 0" rpy="0 0 0" />
+        <geometry>
+          <mesh filename="file://$(find sim)/model/meshes/collision_Link2.stl" />
         </geometry>
       </collision>
@@ -107,11 +107,11 @@
         <origin xyz="0 0 0" rpy="0 0 0" />
         <geometry>
-          <mesh filename="file://$(find rover_system)/model/meshes/Link3.stl" />
-        </geometry>
-      </visual>
-      <collision>
-        <origin xyz="0 0 0" rpy="0 0 0" />
-        <geometry>
-          <mesh filename="file://$(find rover_system)/model/meshes/collision_Link3.stl" />
+          <mesh filename="file://$(find sim)/model/meshes/Link3.stl" />
+        </geometry>
+      </visual>
+      <collision>
+        <origin xyz="0 0 0" rpy="0 0 0" />
+        <geometry>
+          <mesh filename="file://$(find sim)/model/meshes/collision_Link3.stl" />
         </geometry>
       </collision>
@@ -136,11 +136,11 @@
         <origin xyz="0 0 0" rpy="0 0 0" />
         <geometry>
-          <mesh filename="file://$(find rover_system)/model/meshes/Link4.stl" />
-        </geometry>
-      </visual>
-      <collision>
-        <origin xyz="0 0 0" rpy="0 0 0" />
-        <geometry>
-          <mesh filename="file://$(find rover_system)/model/meshes/collision_Link4.stl" />
+          <mesh filename="file://$(find sim)/model/meshes/Link4.stl" />
+        </geometry>
+      </visual>
+      <collision>
+        <origin xyz="0 0 0" rpy="0 0 0" />
+        <geometry>
+          <mesh filename="file://$(find sim)/model/meshes/collision_Link4.stl" />
         </geometry>
       </collision>
@@ -165,11 +165,11 @@
         <origin xyz="0 0 0" rpy="0 0 0" />
         <geometry>
-          <mesh filename="file://$(find rover_system)/model/meshes/Link5.stl" />
-        </geometry>
-      </visual>
-      <collision>
-        <origin xyz="0 0 0" rpy="0 0 0" />
-        <geometry>
-          <mesh filename="file://$(find rover_system)/model/meshes/collision_Link5.stl" />
+          <mesh filename="file://$(find sim)/model/meshes/Link5.stl" />
+        </geometry>
+      </visual>
+      <collision>
+        <origin xyz="0 0 0" rpy="0 0 0" />
+        <geometry>
+          <mesh filename="file://$(find sim)/model/meshes/collision_Link5.stl" />
         </geometry>
       </collision>
@@ -202,5 +202,5 @@
         <origin xyz="0 0 0" rpy="0 0 0" />
         <geometry>
-          <mesh filename="file://$(find rover_system)/model/meshes/finger.stl" />
+          <mesh filename="file://$(find sim)/model/meshes/finger.stl" />
         </geometry>
       </visual>
@@ -223,5 +223,5 @@
         <origin xyz="0 0 0" rpy="0 0 0" />
         <geometry>
-          <mesh filename="file://$(find rover_system)/model/meshes/finger.stl" />
+          <mesh filename="file://$(find sim)/model/meshes/finger.stl" />
         </geometry>
       </visual>

File: sim/model/depth_camera.urdf.xacro (robot description, xacro)
@@ -17,5 +17,5 @@
                 <origin xyz="0 0 0" rpy="0 0 0" />
                 <geometry>
-                    <mesh filename="file://$(find rover_system)/model/meshes/depth_camera.dae"
+                    <mesh filename="file://$(find sim)/model/meshes/depth_camera.dae"
                         scale="1.0 1.0 1.0" />
                 </geometry>

File: sim/model/rover.urdf.xacro (robot description, xacro)
@@ -16,5 +16,5 @@
             <geometry>
                 <mesh
-                    filename="file://$(find rover_system)/model/meshes/Full_Asm_noarm_mast_cam.dae" />
+                    filename="file://$(find sim)/model/meshes/Full_Asm_noarm_mast_cam.dae" />
             </geometry>
         </visual>
@@ -23,5 +23,5 @@
             <geometry>
                 <!-- <mesh
-                    filename="file://$(find rover_system)/model/meshes/Full_Asm_Adjusted.dae" /> -->
+                    filename="file://$(find sim)/model/meshes/Full_Asm_Adjusted.dae" /> -->
                 <box size="0.4 0.6 0.3" />
             </geometry>

File: sim/model/wheel.urdf.xacro (robot description, xacro)
@@ -21,5 +21,5 @@
 				<geometry>
 					<mesh
-						filename="file://$(find rover_system)/model/meshes/WHEEL.dae" />
+						filename="file://$(find sim)/model/meshes/WHEEL.dae" />
 				</geometry>
 			</visual>

Commit message: added dummy legal inertia for arm

File: sim/model/MR_arm.urdf.xacro (robot description, xacro)
@@ -13,5 +13,5 @@
         <mass value="0.1" />
         <origin xyz="0 0 0" rpy="0 0 0" />
-        <inertia ixx="0" ixy="0" ixz="0" iyy="0" iyz="0" izz="0" />
+        <inertia ixx="0.0001" ixy="0" ixz="0" iyy="0.0001" iyz="0" izz="0.0002" />
         <gravity>0</gravity>
         <self_collide>0</self_collide>
@@ -43,5 +43,5 @@
         <mass value="0.1" />
         <origin xyz="0 0 0" rpy="0 0 0" />
-        <inertia ixx="0" ixy="0" ixz="0" iyy="0" iyz="0" izz="0" />
+        <inertia ixx="0.0001" ixy="0" ixz="0" iyy="0.0001" iyz="0" izz="0.0002" />
         <gravity>0</gravity>
         <self_collide>0</self_collide>
@@ -73,5 +73,5 @@
         <mass value="0.1" />
         <origin xyz="0 0 0" rpy="0 0 0" />
-        <inertia ixx="0" ixy="0" ixz="0" iyy="0" iyz="0" izz="0" />
+        <inertia ixx="0.0001" ixy="0" ixz="0" iyy="0.0001" iyz="0" izz="0.0002" />
         <gravity>0</gravity>
         <self_collide>0</self_collide>
@@ -103,5 +103,5 @@
         <mass value="0.1" />
         <origin xyz="0 0 0" rpy="0 0 0" />
-        <inertia ixx="0" ixy="0" ixz="0" iyy="0" iyz="0" izz="0" />
+        <inertia ixx="0.0001" ixy="0" ixz="0" iyy="0.0001" iyz="0" izz="0.0002" />
         <gravity>0</gravity>
         <self_collide>0</self_collide>
@@ -133,5 +133,5 @@
         <mass value="0.1" />
         <origin xyz="0 0 0" rpy="0 0 0" />
-        <inertia ixx="0" ixy="0" ixz="0" iyy="0" iyz="0" izz="0" />
+        <inertia ixx="0.0001" ixy="0" ixz="0" iyy="0.0001" iyz="0" izz="0.0002" />
         <gravity>0</gravity>
         <self_collide>0</self_collide>
@@ -163,5 +163,5 @@
         <mass value="0.1" />
         <origin xyz="0 0 0" rpy="0 0 0" />
-        <inertia ixx="0" ixy="0" ixz="0" iyy="0" iyz="0" izz="0" />
+        <inertia ixx="0.0001" ixy="0" ixz="0" iyy="0.0001" iyz="0" izz="0.0002" />
         <gravity>0</gravity>
         <self_collide>0</self_collide>
@@ -201,5 +201,5 @@
         <mass value="0.1" />
         <origin xyz="0 0 0" rpy="0 0 0" />
-        <inertia ixx="0" ixy="0" ixz="0" iyy="0" iyz="0" izz="0" />
+        <inertia ixx="0.0001" ixy="0" ixz="0" iyy="0.0001" iyz="0" izz="0.0002" />
       </inertial>
       <visual>
@@ -221,5 +221,5 @@
         <mass value="0.1" />
         <origin xyz="0 0 0" rpy="0 0 0" />
-        <inertia ixx="0" ixy="0" ixz="0" iyy="0" iyz="0" izz="0" />
+        <inertia ixx="0.0001" ixy="0" ixz="0" iyy="0.0001" iyz="0" izz="0.0002" />
       </inertial>
       <visual>

File: sim/model/lidar.urdf (robot description, URDF)
Before this commit: robot rplidar_s2, 1 links, 1 joints
Links:
- link lidar_link: geometry visual cylinder length=0.1 radius=0.05

File: sim/model/rover.urdf.xacro (robot description, xacro)
@@ -62,7 +62,7 @@
     </xacro:depth_camera> -->
     <!-- TODO FIXME arm collision crashes gazebo -->
-    <!-- <xacro:MR_arm parent_link="chassis_link">
+    <xacro:MR_arm parent_link="chassis_link">
         <origin xyz="0 -0.28 ${0.37}" rpy="0 0 -1.57079" />
-    </xacro:MR_arm> -->
+    </xacro:MR_arm>
     <!-- Gazebo Plugins -->
     <gazebo>
