Commit message: camera fix

File: sim/model/camera.urdf.xacro (robot description, xacro)
@@ -1,9 +1,9 @@
 <robot xmlns:xacro="http://www.ros.org/wiki/xacro" name="camera">
+    <xacro:property name="M_PI" value="3.14159265" />
     <link name="camera_link" />
     <joint name="camera_to_chassis" type="fixed">
         <parent link="chassis_link" />
         <child link="camera_link" />
-        <origin xyz="0 0 0" rpy="0 0 0" />
-        <pose>0.05 0.05 0.05 0 0 0</pose>
+        <origin xyz="0 0 0" rpy="0 0 ${M_PI/2}" />
         <!-- <collision name="collision">
             <geometry>
@@ -12,5 +12,5 @@
                 </box>
             </geometry>
-        </collision>
+        </collision> -->
         <visual name="visual">
             <geometry>
@@ -19,5 +19,5 @@
                 </box>
             </geometry>
-        </visual> -->
+        </visual>
     </joint>
     <gazebo reference="camera_link">

Commit message: fix camera rotation

File: sim/model/camera.urdf.xacro (robot description, xacro)
@@ -5,18 +5,24 @@
         <parent link="chassis_link" />
         <child link="camera_link" />
-        <origin xyz="0 0 0" rpy="0 0 ${M_PI/2}" />
+        <origin xyz="0 0 0" rpy="0 0 -${M_PI/2}" />
+        <!-- Collision block commented out for now -->
         <!-- <collision name="collision">
             <geometry>
-                <box>
-                    <size>0.1 0.1 0.1</size>
-                </box>
+                <cylinder>
+                    <radius>0.05</radius>
+                    <length>0.2</length>
+                </cylinder>
             </geometry>
         </collision> -->
-        <visual name="visual">
+        <visual name="camera_visual">
             <geometry>
-                <box>
-                    <size>0.1 0.1 0.1</size>
-                </box>
+                <cylinder>
+                    <radius>1</radius>
+                    <length>2</length>
+                </cylinder>
             </geometry>
+            <material>
+                <color rgba="0 0 1 1"/> <!-- Blue color for the camera -->
+            </material>
         </visual>
     </joint>
@@ -42,4 +48,5 @@
     </gazebo>
     <gazebo>
+        <!-- Plugin for rendering engine, commented out for now -->
         <!-- <plugin
             filename="ignition-gazebo-sensors-system"
