Commit message: sensors WIP

File: sim/model/depth_camera.urdf.xacro (robot description, xacro)
@@ -1,34 +1,37 @@
-<?xml version="1.0"?>
-<robot name="kinect" xmlns:xacro="http://ros.org/wiki/xacro">
-    <xacro:macro name="depth_camera" params="parent_link *joint_pose">
+<sdf version="1.9">
+    <model name="kinect">
         <link name="kinect_link">
             <inertial>
-                <mass value="0.1" />
-                <origin xyz="0 0 0" rpy="0 0 0" />
-                <inertia ixx="0" ixy="0" ixz="0" iyy="0" iyz="0" izz="0" />
+                <mass>0.1</mass>
+                <inertia>
+                    <ixx>0</ixx>
+                    <ixy>0</ixy>
+                    <ixz>0</ixz>
+                    <iyy>0</iyy>
+                    <iyz>0</iyz>
+                    <izz>0</izz>
+                </inertia>
             </inertial>
             <collision name="kinect_collision">
-                <origin xyz="0 0 0" rpy="0 0 0" />
+                <pose>0 0 0 0 0 0</pose>
                 <geometry>
-                    <box size="0.073000 0.276000 0.072000" />
+                    <box>
+                        <size>0.073 0.276 0.072</size>
+                    </box>
                 </geometry>
             </collision>
             <visual name="kinect_visual">
-                <origin xyz="0 0 0" rpy="0 0 0" />
+                <pose>0 0 0 0 0 0</pose>
                 <geometry>
-                    <mesh filename="file://$(find sim)/model/meshes/depth_camera.dae"
-                        scale="1.0 1.0 1.0" />
+                    <mesh>
+                        <uri>file://meshes/depth_camera.dae</uri>
+                        <scale>1.0 1.0 1.0</scale>
+                    </mesh>
                 </geometry>
             </visual>
-        </link>
-        <joint name="depth_camera_joint" type="fixed">
-            <parent link="${parent_link}" />
-            <child link="kinect_link" />
-            <xacro:insert_block name="joint_pose" />
-        </joint>
-        <gazebo reference="kinect_link">
-            <sensor name="camera" type="depth">
+            <sensor name="camera" type="depth_camera">
+                <pose>0 0 0 0 0 0</pose>
                 <update_rate>20</update_rate>
-                <camera>
+                <depth_camera>
                     <horizontal_fov>1.047198</horizontal_fov>
                     <image>
@@ -41,33 +44,20 @@
                         <far>3</far>
                     </clip>
-                </camera>
-                <plugin name="camera_plugin" filename="libgazebo_ros_openni_kinect.so">
-                    <baseline>0.2</baseline>
-                    <alwaysOn>true</alwaysOn>
-                    <!-- Keep this zero, update_rate in the parent <sensor> tag
-                    will control the frame rate. -->
-                    <updateRate>0.0</updateRate>
-                    <cameraName>camera_ir</cameraName>
-                    <imageTopicName>/camera/color/image_raw</imageTopicName>
-                    <cameraInfoTopicName>/camera/color/camera_info</cameraInfoTopicName>
-                    <depthImageTopicName>/camera/depth/image_raw</depthImageTopicName>
-                    <depthImageCameraInfoTopicName>/camera/depth/camera_info</depthImageCameraInfoTopicName>
-                    <pointCloudTopicName>/camera/depth/points</pointCloudTopicName>
-                    <frameName>camera_link</frameName>
-                    <pointCloudCutoff>0.5</pointCloudCutoff>
-                    <pointCloudCutoffMax>3.0</pointCloudCutoffMax>
-                    <distortionK1>0</distortionK1>
-                    <distortionK2>0</distortionK2>
-                    <distortionK3>0</distortionK3>
-                    <distortionT1>0</distortionT1>
-                    <distortionT2>0</distortionT2>
-                    <CxPrime>0</CxPrime>
-                    <Cx>0</Cx>
-                    <Cy>0</Cy>
-                    <focalLength>0</focalLength>
-                    <hackBaseline>0</hackBaseline>
+                </depth_camera>
+                <plugin
+                    name="ignition::sensors::DepthCameraSensor"
+                    filename="ignition-gazebo-depth-camera-system">
+                    <topic>/camera/depth/image_raw</topic>
+                    <camera_info_topic>/camera/depth/camera_info</camera_info_topic>
+                    <point_cloud_topic>/camera/depth/points</point_cloud_topic>
+                    <frame_id>camera_link</frame_id>
                 </plugin>
             </sensor>
-        </gazebo>
-    </xacro:macro>
-</robot>
+        </link>
+        <joint name="depth_camera_joint" type="fixed">
+            <parent>parent_link</parent>
+            <child>kinect_link</child>
+            <pose>0 0 0 0 0 0</pose>
+        </joint>
+    </model>
+</sdf>

File: sim/model/rover.urdf.xacro (robot description, xacro)
@@ -5,8 +5,11 @@
     <xacro:property name="wheel_z_offset" value="${-0.060752 + 0.1}" />
     <!-- Part Includes - Payload, Sensors, Etc.. -->
-    <xacro:include filename="$(find rover_system)/model/wheel.urdf.xacro" />
-    <!-- <xacro:include filename="$(find rover_system)/model/depth_camera.urdf.xacro" />a -->
-    <xacro:include filename="$(find rover_system)/model/MR_arm.urdf.xacro" />
-    <xacro:include filename="$(find rover_system)/model/imu.urdf" />
+    <xacro:include filename="$(find sim)/model/wheel.urdf.xacro" />
+    <xacro:include filename="$(find sim)/model/depth_camera.urdf.xacro" />
+    <xacro:include filename="$(find sim)/model/MR_arm.urdf.xacro" />
+    <xacro:include filename="$(find sim)/model/imu.urdf" />
+    <xacro:include filename="$(find sim)/model/lidar.urdf" />
+    <xacro:include filename="$(find sim)/model/camera.urdf.xacro" />
+    <!-- <xacro:include filename="$(find sim)/model/thermal_camera.urdf" /> -->
     <!-- Robot Definition -->
     <link name="base_link" />
@@ -59,7 +62,7 @@
     </xacro:depth_camera> -->
     <!-- TODO FIXME arm collision crashes gazebo -->
-    <xacro:MR_arm parent_link="chassis_link">
+    <!-- <xacro:MR_arm parent_link="chassis_link">
         <origin xyz="0 -0.28 ${0.37}" rpy="0 0 -1.57079" />
-    </xacro:MR_arm>
+    </xacro:MR_arm> -->
     <!-- Gazebo Plugins -->
     <gazebo>

Commit message: feat: converted depth_camera to xacro and added bridges

File: sim/model/depth_camera.urdf.xacro (robot description, xacro)
@@ -1,63 +1,58 @@
-<sdf version="1.9">
-    <model name="kinect">
-        <link name="kinect_link">
-            <inertial>
-                <mass>0.1</mass>
-                <inertia>
-                    <ixx>0</ixx>
-                    <ixy>0</ixy>
-                    <ixz>0</ixz>
-                    <iyy>0</iyy>
-                    <iyz>0</iyz>
-                    <izz>0</izz>
-                </inertia>
-            </inertial>
-            <collision name="kinect_collision">
-                <pose>0 0 0 0 0 0</pose>
-                <geometry>
-                    <box>
-                        <size>0.073 0.276 0.072</size>
-                    </box>
-                </geometry>
-            </collision>
-            <visual name="kinect_visual">
-                <pose>0 0 0 0 0 0</pose>
-                <geometry>
-                    <mesh>
-                        <uri>file://meshes/depth_camera.dae</uri>
-                        <scale>1.0 1.0 1.0</scale>
-                    </mesh>
-                </geometry>
-            </visual>
-            <sensor name="camera" type="depth_camera">
-                <pose>0 0 0 0 0 0</pose>
-                <update_rate>20</update_rate>
-                <depth_camera>
-                    <horizontal_fov>1.047198</horizontal_fov>
-                    <image>
-                        <width>640</width>
-                        <height>480</height>
-                        <format>R8G8B8</format>
-                    </image>
-                    <clip>
-                        <near>0.05</near>
-                        <far>3</far>
-                    </clip>
-                </depth_camera>
-                <plugin
-                    name="ignition::sensors::DepthCameraSensor"
-                    filename="ignition-gazebo-depth-camera-system">
-                    <topic>/camera/depth/image_raw</topic>
-                    <camera_info_topic>/camera/depth/camera_info</camera_info_topic>
-                    <point_cloud_topic>/camera/depth/points</point_cloud_topic>
-                    <frame_id>camera_link</frame_id>
-                </plugin>
-            </sensor>
-        </link>
-        <joint name="depth_camera_joint" type="fixed">
-            <parent>parent_link</parent>
-            <child>kinect_link</child>
-            <pose>0 0 0 0 0 0</pose>
-        </joint>
-    </model>
-</sdf>
+<robot xmlns:xacro="http://ros.org/wiki/xacro">
+  <xacro:macro name="depth_camera" params="parent_link origin_xyz origin_rpy">
+    <!-- Joint connecting camera to parent -->
+    <joint name="depth_camera_joint" type="fixed">
+      <parent link="${parent_link}" />
+      <child link="kinect_link" />
+      <origin xyz="${origin_xyz}" rpy="${origin_rpy}" />
+    </joint>
+    <!-- Camera Link -->
+    <link name="kinect_link">
+      <inertial>
+        <mass value="0.1" />
+        <inertia ixx="0" ixy="0" ixz="0" iyy="0" iyz="0" izz="0" />
+      </inertial>
+      <collision name="kinect_collision">
+        <origin xyz="0 0 0" rpy="0 0 0" />
+        <geometry>
+          <box size="0.073 0.276 0.072" />
+        </geometry>
+      </collision>
+      <visual name="kinect_visual">
+        <origin xyz="0 0 0" rpy="0 0 0" />
+        <geometry>
+          <mesh filename="file://$(find sim)/model/meshes/depth_camera.dae" />
+        </geometry>
+      </visual>
+    </link>
+    <!-- Gazebo Sensor Plugin -->
+    <gazebo reference="kinect_link">
+      <sensor name="depth_camera" type="depth_camera">
+        <update_rate>20</update_rate>
+        <visualize>true</visualize>
+        <always_on>true</always_on>
+        <pose>0 0 0 0 0 0</pose>
+        <depth_camera>
+          <horizontal_fov>1.047198</horizontal_fov>
+          <image>
+            <width>640</width>
+            <height>480</height>
+            <format>R8G8B8</format>
+          </image>
+          <clip>
+            <near>0.05</near>
+            <far>3.0</far>
+          </clip>
+        </depth_camera>
+        <!-- Topic and Frame Info -->
+        <topic>/camera/depth/image_raw</topic>
+        <camera_info_topic>/camera/depth/camera_info</camera_info_topic>
+        <point_cloud_topic>/camera/depth/points</point_cloud_topic>
+        <frame_id>kinect_link</frame_id>
+        <plugin name="gazebo_ros_depth_camera" filename="libgazebo_ros_depth_camera.so">
+          <frame_name>kinect_link</frame_name>
+        </plugin>
+      </sensor>
+    </gazebo>
+  </xacro:macro>
+</robot>

File: sim/model/rover.urdf.xacro (robot description, xacro)
@@ -58,7 +58,7 @@
         <origin xyz="-0.5125 0.306875 ${wheel_z_offset}" rpy="0 ${M_PI/2} 0" />
     </xacro:wheel>
-    <!-- <xacro:depth_camera parent_link="chassis_link">
-        <origin xyz="0 -0.41 0.32" rpy="0 0 -1.57079" />
-    </xacro:depth_camera> -->
+    <xacro:depth_camera parent_link="chassis_link"
+                    origin_xyz="0 -0.8 0.32"
+                    origin_rpy="0 0 -1.5708" />
     <!-- TODO FIXME arm collision crashes gazebo -->
     <xacro:MR_arm parent_link="chassis_link">
