Commit message: WIP: Cleaned Up Code and Added Fix to Import Rover into Sim

File: pybullet_drive_sim/urdf/ROVER_DRIVE.urdf (robot description, URDF)
Before this commit: robot ROVER_DRIVE, 16 links, 15 joints
Joints:
- joint Left Link Rocker: axis 0 0 0 -> 0 0 1
- joint Right Link Rocker: axis 0 0 0 -> 0 0 1
