Commit message: Fix: Rover moves correctly now with skid steering

File: sim/halley/halley_rover.urdf (robot description, URDF)
Before this commit: robot halley_rover, 7 links, 6 joints
Joints:
- joint wheel_1_joint: axis 0.014692 0 0.99989 -> -0.014692 0 -0.99989
- joint wheel_2_joint: axis 0.014692 0 0.99989 -> -0.014692 0 -0.99989
